File: PeltierDrive.kicad_pcb (KiCad board)
At the start: 2 copper layers, 28 parts, among them U2 MCP4725xxx-xCH, U4 MCP3422Axx-xSN

Commit message: commponents placed roughly
Parts:
- added C15: 10u, Capacitor_SMD:C_0805_2012Metric_Pad1.18x1.45mm_HandSolder, F.Cu at (46.6, 112.7)
- added C16: 10u, Capacitor_SMD:C_0805_2012Metric_Pad1.18x1.45mm_HandSolder, F.Cu at (82.2, 111.8)
- added J1: V in, TerminalBlock_MetzConnect:TerminalBlock_MetzConnect_Type086_RT03402HBLC_1x02_P3.81mm_Horizontal, F.Cu at (65.4, 103.8)
- added J2: V out, TerminalBlock_MetzConnect:TerminalBlock_MetzConnect_Type086_RT03402HBLC_1x02_P3.81mm_Horizontal, F.Cu at (52.0, 104.0)
- added J3: socket NTC, TerminalBlock_MetzConnect:TerminalBlock_MetzConnect_Type086_RT03402HBLC_1x02_P3.81mm_Horizontal, F.Cu at (75.6, 103.8)
- added J4: Conn_01x06_Socket, Connector_PinHeader_2.54mm:PinHeader_1x06_P2.54mm_Horizontal, F.Cu at (89.0, 108.5)
- added L1: 22uH, Inductor_SMD:L_12x12mm_H8mm, F.Cu at (52.0, 123.0)
- added R11: 3K3, Resistor_SMD:R_0603_1608Metric_Pad0.98x0.95mm_HandSolder, F.Cu at (89.0, 102.0)
- added R12: 3K3, Resistor_SMD:R_0603_1608Metric_Pad0.98x0.95mm_HandSolder, F.Cu at (89.0, 104.0)
- added U1: AOZ1284PI, Package_SO:SOIC-8-1EP_3.9x4.9mm_P1.27mm_EP2.71x3.7mm, F.Cu at (64.1, 120.3)
- added U3: AP2127N-2.8, Package_TO_SOT_SMD:SOT-23, F.Cu at (78.4, 111.8)
- C1, C10, C11, C12, C13, C14, C2, C3, C4, C5, C6, C7, C8, C9: footprint Capacitor_SMD:C_0603_1608Metric_Pad1.08x0.95mm_HandSolder -> Capacitor_SMD:C_0805_2012Metric_Pad1.18x1.45mm_HandSolder
- moved C9 97.8 mm to (46.6, 110.2), turned to 180 degrees
- moved R9 94.7 mm to (56.5, 106.3), turned to -90 degrees
- moved R8 94.5 mm to (56.5, 102.9), turned to -90 degrees
- moved C8 94.5 mm to (51.7, 112.7)
- moved D2 94.4 mm to (66.7, 112.7), turned to -90 degrees
- moved R4 90.3 mm to (61.6, 125.8), turned to -90 degrees
- moved C3 89.0 mm to (51.4, 110.2)
- moved R3 88.9 mm to (64.1, 125.8), turned to -90 degrees
- moved C7 87.3 mm to (61.4, 115.2), turned to 180 degrees
- moved R5 87.0 mm to (76.0, 125.8), turned to -90 degrees
- moved C2 85.9 mm to (59.0, 118.8), turned to 90 degrees
- moved R6 85.2 mm to (74.0, 121.0)
- moved R2 83.9 mm to (71.0, 125.8), turned to -90 degrees
- moved D1 83.5 mm to (56.5, 111.4), turned to 90 degrees
- moved R7 82.9 mm to (73.0, 116.0), turned to 90 degrees
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Connections:
- R10 pad 1: +3.3V -> +2V8
Routing:
- net Net-(J3-Pin_1): track 0.00 -> 11.2 mm
Other:
- board outline added: 60 x 30 mm

Commit message: layout completed
Parts:
- added C17: 2.2n, Capacitor_SMD:C_0603_1608Metric_Pad1.08x0.95mm_HandSolder, F.Cu at (73.0, 120.4)
- added C18: 2.2n, Capacitor_SMD:C_0805_2012Metric_Pad1.18x1.45mm_HandSolder, F.Cu at (69.0, 127.5)
- added J5: Conn_01x03_Pin, Connector_PinHeader_2.54mm:PinHeader_1x03_P2.54mm_Vertical, F.Cu at (43.0, 115.3)
- J1, J2, J3: footprint TerminalBlock_MetzConnect:TerminalBlock_MetzConnect_Type086_RT03402HBLC_1x02_P3.81mm_Horizontal -> TerminalBlock_MetzConnect:TerminalBlock_MetzConnect_Type094_RT03502HBLU_1x02_P5.00mm_Horizontal
- R8, R9: footprint Resistor_SMD:R_0603_1608Metric_Pad0.98x0.95mm_HandSolder -> Resistor_SMD:R_0805_2012Metric_Pad1.20x1.40mm_HandSolder
- moved C14 17.8 mm to (85.0, 120.5), turned to 180 degrees
- moved R5 14.5 mm to (90.4, 124.5), turned to 0 degrees
- moved J3 6.00 mm to (81.5, 104.6), turned to 180 degrees
- moved R10 5.80 mm to (84.0, 113.0), turned to 0 degrees
- moved J1 5.17 mm to (70.5, 104.6)
- moved C3 4.32 mm to (55.5, 111.5)
- moved C8 4.02 mm to (55.5, 114.0)
- moved R6 4.00 mm to (74.1, 117.0)
- moved C1 3.56 mm to (64.0, 112.5)
- moved R8 3.54 mm to (60.0, 103.5), turned to 0 degrees
- moved D1 3.54 mm to (60.0, 112.0)
- moved C6 3.53 mm to (64.0, 115.0)
- moved R9 3.51 mm to (60.0, 106.0), turned to 180 degrees
- moved C7 3.51 mm to (64.0, 117.5)
- moved C13 3.37 mm to (81.0, 119.5), turned to -90 degrees
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Connections:
- net Net-(D1-K) renamed LX
- net Net-(D2-K) renamed V_{IN}
- C14 pad 1: Net-(J3-Pin_1) -> V_{NTC}
- C15 pad 1: Net-(J2-Pin_2) -> V_{OUT}
- C3 pad 1: Net-(J2-Pin_2) -> V_{OUT}
- C8 pad 1: Net-(J2-Pin_2) -> V_{OUT}
- C9 pad 1: Net-(J2-Pin_2) -> V_{OUT}
- J2 pad 2: Net-(J2-Pin_2) -> V_{OUT}
- J3 pad 1: Net-(J3-Pin_1) -> GND
- J3 pad 2: GND -> V_{NTC}
- L1 pad 2: Net-(J2-Pin_2) -> V_{OUT}
- R1 pad 1: Net-(J2-Pin_2) -> Net-(U1-FB)
- R1 pad 2: Net-(U1-FB) -> V_{OUT}
- R10 pad 2: Net-(J3-Pin_1) -> V_{NTC}
- U4 pad 1: Net-(J3-Pin_1) -> V_{NTC}
Routing:
- net Net-(J2-Pin_1): track 0.00 -> 76.8 mm, vias 0 -> 2
- net Net-(U4-CH2-): track 0.00 -> 70.9 mm
- net GND: track 0.00 -> 66.6 mm, vias 0 -> 65
- net SCL: track 0.00 -> 48.1 mm, vias 0 -> 2
- net Vctrl: track 0.00 -> 46.1 mm, vias 0 -> 1
- net V_{OUT}: track 0.00 -> 45.3 mm, vias 0 -> 1
- net SDA: track 0.00 -> 39.9 mm, vias 0 -> 2
- net EN: track 0.00 -> 32.1 mm, vias 0 -> 1
- net +3.3V: track 0.00 -> 24.2 mm, vias 0 -> 7
- net V_{NTC}: track 0.00 -> 23.7 mm
- net LX: track 0.00 -> 22.3 mm
- net Net-(D2-A): track 0.00 -> 21.0 mm, vias 0 -> 6
- net Net-(U1-FB): track 0.00 -> 12.2 mm
- net Net-(J3-Pin_1): track 11.2 -> 0.00 mm
- net Net-(U1-SS): track 0.00 -> 8.95 mm, vias 0 -> 2
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- added copper zone on In2.Cu, net +3.3V
- added copper zone on B.Cu, net GND
- added copper zone on F.Cu, net GND
- added copper zone on In1.Cu, net GND
- added copper zone on F.Cu, net V_{IN}
- added copper zone on F.Cu, net V_{OUT}
Other:
- outline, holes or cut-outs redrawn
- copper layers 2 -> 4
- board text added: "LG"
- board text added: "Łukasz G PelterDrive V1.0"

Commit message: pushed PCB to manufacturing
Parts:
- added C19: 10u, Capacitor_SMD:C_0805_2012Metric_Pad1.18x1.45mm_HandSolder, F.Cu at (92.0, 127.0)
- C2: footprint Capacitor_SMD:C_0805_2012Metric_Pad1.18x1.45mm_HandSolder -> Capacitor_SMD:C_0603_1608Metric_Pad1.08x0.95mm_HandSolder
- moved R5 1.09 mm to (89.5, 125.1), turned to -90 degrees
- moved R10 1.00 mm to (84.0, 114.0)
- moved C2 0.50 mm to (60.5, 120.5)
Routing:
- net LX: track 22.3 -> 25.1 mm
- net GND: track 66.6 -> 68.1 mm, vias 65 -> 68
- net +2V8: track 6.47 -> 7.58 mm
- net EN: track 32.1 -> 31.3 mm
