File: PeltierDrive.kicad_sch (KiCad schematic)
At the start: 34 parts, among them J1 V in, J2 V out, J3 socket NTC, J4 Conn_01x06_Socket, U1 AOZ1284PI, U2 MCP4725xxx-xCH, U4 MCP3422Axx-xSN

Commit message: commponents placed roughly
Parts:
- added C15, C16: 10u, Capacitor_SMD:C_0805_2012Metric_Pad1.18x1.45mm_HandSolder, symbol Device:C
- added R11, R12: 3K3, Resistor_SMD:R_0603_1608Metric_Pad0.98x0.95mm_HandSolder, symbol Device:R
- added U3: AP2127N-2.8, Package_TO_SOT_SMD:SOT-23, symbol Regulator_Linear:AP2127N-2.8
- C1, C10, C11, C12, C13, C14, C2, C3, C4, C5, C6, C7, C8, C9: footprint Capacitor_SMD:C_0603_1608Metric_Pad1.08x0.95mm_HandSolder -> Capacitor_SMD:C_0805_2012Metric_Pad1.18x1.45mm_HandSolder
- J1, J2, J3: footprint (none) -> TerminalBlock_MetzConnect:TerminalBlock_MetzConnect_Type086_RT03402HBLC_1x02_P3.81mm_Horizontal
- J4: footprint (none) -> Connector_PinHeader_2.54mm:PinHeader_1x06_P2.54mm_Horizontal
- L1: footprint (none) -> Inductor_SMD:L_12x12mm_H8mm
Connections:
- net +3.3V: now also R11.1, R12.1, U3.3 (VI); no longer R10.1
- net GND: now also C15.2, C16.2, U3.1 (GND)
- net SCL: now also R11.2
- net SDA: now also R12.2
- net at C3.1, C8.1, C9.1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: now also C15.1
- new net +2V8: C16.1, R10.1, U3.2 (VO)
Other:
- moved on the sheet: C13

Commit message: layout completed
Parts:
- added C17: 2.2n, Capacitor_SMD:C_0603_1608Metric_Pad1.08x0.95mm_HandSolder, symbol Device:C
- added C18: 2.2n, Capacitor_SMD:C_0805_2012Metric_Pad1.18x1.45mm_HandSolder, symbol Device:C
- added J5: Conn_01x03_Pin, Connector_PinHeader_2.54mm:PinHeader_1x03_P2.54mm_Vertical, symbol Connector:Conn_01x03_Pin
- J1, J2, J3: footprint TerminalBlock_MetzConnect:TerminalBlock_MetzConnect_Type086_RT03402HBLC_1x02_P3.81mm_Horizontal -> TerminalBlock_MetzConnect:TerminalBlock_MetzConnect_Type094_RT03502HBLU_1x02_P5.00mm_Horizontal
- R8, R9: footprint Resistor_SMD:R_0603_1608Metric_Pad0.98x0.95mm_HandSolder -> Resistor_SMD:R_0805_2012Metric_Pad1.20x1.40mm_HandSolder
Connections:
- net GND: now also J3.1 (Pin_1), C18.2, J5.3 (Pin_3); no longer J3.2 (Pin_2)
- net Vctrl: now also J5.2 (Pin_2)
- net V_{OUT}: now reaches C15.1, C3.1, C8.1, C9.1, J2.2 (Pin_2), L1.2
- net V_{OUT}: now also R1.2, C17.1, J5.1 (Pin_1); no longer R1.1
- net V_{NTC}: now reaches C14.1, R10.2, U4.1 (CH1+)
- net V_{NTC}: now also J3.2 (Pin_2); no longer J3.1 (Pin_1)
- net at R2.1, R6.1, U1.6 (FB): now also R1.1, C17.2; no longer R1.2
- net at C5.1, U1.5 (COMP): now also C18.1
- net V_{IN}: now reaches C1.1, C6.1, C7.1, D2.1 (K), U1.9 (VIN)
- net LX: now reaches C2.2, D1.1 (K), L1.1, U1.1 (LX)

Commit message: pushed PCB to manufacturing
Parts:
- added C19: 10u, Capacitor_SMD:C_0805_2012Metric_Pad1.18x1.45mm_HandSolder, symbol Device:C
- C2: footprint Capacitor_SMD:C_0805_2012Metric_Pad1.18x1.45mm_HandSolder -> Capacitor_SMD:C_0603_1608Metric_Pad1.08x0.95mm_HandSolder
- D1, D2: value SS34 -> PMEG4050CEPX
- R1: value 100k -> 27k
- R8: value 0.01R -> 0.02R
Connections:
- net at J2.1 (Pin_1), R8.1, U4.7 (CH2+): now also C19.1
- net at R8.2, R9.1, U4.8 (CH2-): now also C19.2
Changed lines of the file:
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@@
 	)
 	(junction
+		(at 241.3 100.33)
+		(diameter 0)
+		(color 0 0 0 0)
+	)
+	(junction
+		(at 241.3 111.76)
+		(diameter 0)
+		(color 0 0 0 0)
+	)
+	(junction
 		(at 224.79 101.6)
 		(diameter 0)
@@
 	(wire
 		(pts
+			(xy 241.3 100.33) (xy 241.3 101.6)
+		)
+		(stroke
+			(width 0)
+			(type default)
+		)
+	)
+	(wire
+		(pts
 			(xy 111.76 156.21) (xy 111.76 157.48)
 		)
@@
 	(wire
 		(pts
+			(xy 241.3 100.33) (xy 245.11 100.33)
+		)
+		(stroke
+			(width 0)
+			(type default)
+		)
+	)
+	(wire
+		(pts
 			(xy 187.96 97.79) (xy 177.8 97.79)
 		)
@@
 	(wire
 		(pts
+			(xy 241.3 109.22) (xy 241.3 111.76)
+		)
+		(stroke
+			(width 0)
+			(type default)
+		)
+	)
+	(wire
+		(pts
 			(xy 50.8 68.58) (xy 50.8 69.85)
 		)
@@
 	(wire
 		(pts
-			(xy 238.76 100.33) (xy 245.11 100.33)
+			(xy 238.76 100.33) (xy 241.3 100.33)
 		)
 		(stroke
@@
 			)
 		)
-		(property "Value" "100k"
+		(property "Value" "27k"
 			(at 190.5 101.6001 0)
 			(effects
@@
 			)
 		)
-		(property "Value" "SS34"
+		(property "Value" "PMEG4050CEPX"
 			(at 53.6575 88.9 0)
 			(effects
@@
 					(size 1.27 1.27)
 				)
+				(hide yes)
 			)
 		)
@@
 			)
 		)
-		(property "Datasheet" "https://www.vishay.com/docs/88751/ss32.pdf"
+		(property "Datasheet" "https://www.digikey.nl/en/products/detail/nexperia-usa-inc/PMEG4050CEPX/26266246"
 			(at 53.34 92.71 0)
 			(effects
@@
 			)
 		)
-		(property "Description" "40V 3A Schottky Diode, SMA"
+		(property "Description" "40V 5A Schottky Diode, SMA (SOD-128/CFP5)"
 			(at 53.34 92.71 0)
 			(effects
@@
 			)
 		)
-		(property "Value" "0.01R"
+		(property "Value" "0.02R"
 			(at 247.65 109.2199 0)
 			(effects
@@
 			)
 		)
-		(property "Footprint" "Capacitor_SMD:C_0805_2012Metric_Pad1.18x1.45mm_HandSolder"
+		(property "Footprint" "Capacitor_SMD:C_0603_1608Metric_Pad1.08x0.95mm_HandSolder"
 			(at 153.3652 97.79 0)
 			(effects
@@
 			)
 		)
-		(property "Value" "SS34"
+		(property "Value" "PMEG4050CEPX"
 			(at 165.1 102.5524 90)
 			(effects
@@
 				)
 				(justify left)
+				(hide yes)
 			)
 		)
@@
 			)
 		)
-		(property "Datasheet" "https://www.vishay.com/docs/88751/ss32.pdf"
+		(property "Datasheet" "https://www.digikey.nl/en/products/detail/nexperia-usa-inc/PMEG4050CEPX/26266246"
 			(at 162.56 101.6 0)
 			(effects
@@
 			)
 		)
-		(property "Description" "40V 3A Schottky Diode, SMA"
+		(property "Description" "40V 5A Schottky Diode, SMA (SOD-128/CFP5)"
 			(at 162.56 101.6 0)
 			(effects
@@
 	)
 	(symbol
+		(lib_id "Device:C")
+		(at 241.3 105.41 0)
+		(unit 1)
+		(exclude_from_sim no)
+		(in_bom yes)
+		(on_board yes)
+		(dnp no)
+		(fields_autoplaced yes)
+		(property "Reference" "C19"
+			(at 245.11 104.1399 0)
+			(effects
+				(font
+					(size 1.27 1.27)
+				)
+				(justify left)
+			)
+		)
+		(property "Value" "10u"
+			(at 245.11 106.6799 0)
+			(effects
+				(font
+					(size 1.27 1.27)
+				)
+				(justify left)
+			)
+		)
+		(property "Footprint" "Capacitor_SMD:C_0805_2012Metric_Pad1.18x1.45mm_HandSolder"
+			(at 242.2652 109.22 0)
+			(effects
+				(font
+					(size 1.27 1.27)
+				)
+				(hide yes)
+			)
+		)
+		(property "Datasheet" "~"
+			(at 241.3 105.41 0)
+			(effects
+				(font
+					(size 1.27 1.27)
+				)
+				(hide yes)
+			)
+		)
+		(property "Description" "Unpolarized capacitor"
+			(at 241.3 105.41 0)
+			(effects
+				(font
+					(size 1.27 1.27)
+				)
+				(hide yes)
+			)
+		)
+		(pin "2"
+		)
+		(pin "1"
+		)
+		(instances
+			(project "PeltierDrive"
+				(path "/e47fbdb3-9567-4c4b-b53e-aa89db06e06a"
+					(reference "C19")
+					(unit 1)
+				)
+			)
+		)
+	)
+	(symbol
 		(lib_id "Connector:Conn_01x02_Socket")
 		(at 39.37 95.25 180)
@@
 			)
 		)
-		(property "Datasheet" "~"
+		(property "Datasheet" "https://www.tme.eu/Document/68e226b9b1c2983a3b0686929d941e18/PCS.pdf"
 			(at 173.99 97.79 0)
 			(effects
@@
 			)
 		)
-		(property "Description" "Inductor"
+		(property "Description" "PCS129MT220"
 			(at 173.99 97.79 0)
 			(effects
