File: KiCad/PeltierDrive.kicad_pcb (KiCad board)
At the start: 4 copper layers, 60 x 30 mm, 43 parts, among them J1 V in, J2 V out, J3 socket NTC, J4 Conn_01x06_Socket, J5 Conn_01x03_Pin, U1 AOZ1284PI, U2 MCP4725xxx-xCH, U3 AP2127N-2.8, U4 MCP3422Axx-xSN

Commit message: bom updats after the PCB assembly
Parts:
- D1, D2: value SS34 -> PMEG3050CEP
- R1: value 100k -> 68k
- R10: value 2k -> 20k
- R11, R12: value 3K3 -> 10K
- R8: value 0.01R -> 0.02R
- U3: value AP2127N-2.8 -> TPS7A528PDBZR
Changed lines of the file:
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@@
 			)
 		)
-		(property "Value" "3K3"
+		(property "Value" "10K"
 			(at 0 1.43 0)
 			(layer "F.Fab")
@@
 			)
 		)
-		(property "Value" "2k"
+		(property "Value" "20k"
 			(at 0 1.43 0)
 			(layer "F.Fab")
@@
 			)
 		)
-		(property "Value" "100k"
+		(property "Value" "68k"
 			(at 0.5 0.43 90)
 			(layer "F.Fab")
@@
 			)
 		)
-		(property "Value" "SS34"
+		(property "Value" "PMEG3050CEP"
 			(at -1.3 1.43 90)
 			(layer "F.Fab")
@@
 			)
 		)
-		(property "Datasheet" "https://www.vishay.com/docs/88751/ss32.pdf"
+		(property "Datasheet" "https://www.digikey.nl/en/products/detail/nexperia-usa-inc/PMEG4050CEPX/26266246"
 			(at 0 0 90)
 			(unlocked yes)
@@
 			)
 		)
-		(property "Description" "40V 3A Schottky Diode, SMA"
+		(property "Description" "40V 5A Schottky Diode, SMA (SOD-128/CFP5)"
 			(at 0 0 90)
 			(unlocked yes)
@@
 			)
 		)
-		(property "Value" "AP2127N-2.8"
+		(property "Value" "TPS7A528PDBZR"
 			(at 0 2.4 0)
 			(layer "F.Fab")
@@
 			)
 		)
-		(property "Value" "3K3"
+		(property "Value" "10K"
 			(at 0 1.43 0)
 			(layer "F.Fab")
@@
 			)
 		)
-		(property "Value" "SS34"
+		(property "Value" "PMEG3050CEP"
 			(at 0 2.6 90)
 			(layer "F.Fab")
@@
 			)
 		)
-		(property "Datasheet" "https://www.vishay.com/docs/88751/ss32.pdf"
+		(property "Datasheet" "https://www.digikey.nl/en/products/detail/nexperia-usa-inc/PMEG4050CEPX/26266246"
 			(at 0 0 270)
 			(unlocked yes)
@@
 			)
 		)
-		(property "Description" "40V 3A Schottky Diode, SMA"
+		(property "Description" "40V 5A Schottky Diode, SMA (SOD-128/CFP5)"
 			(at 0 0 270)
 			(unlocked yes)
@@
 			)
 		)
-		(property "Value" "0.01R"
+		(property "Value" "0.02R"
 			(at 0 1 0)
 			(layer "F.Fab")
@@
 			)
 		)
-		(property "Datasheet" "~"
+		(property "Datasheet" "https://www.tme.eu/Document/68e226b9b1c2983a3b0686929d941e18/PCS.pdf"
 			(at 0 0 90)
 			(unlocked yes)
@@
 			)
 		)
-		(property "Description" "Inductor"
+		(property "Description" "PCS129MT220"
 			(at 0 0 90)
 			(unlocked yes)
