File: KiCad/PeltierDrive.kicad_sch (KiCad schematic)
At the start: 43 parts, among them J1 V in, J2 V out, J3 socket NTC, J4 Conn_01x06_Socket, J5 Conn_01x03_Pin, U1 AOZ1284PI, U2 MCP4725xxx-xCH, U3 AP2127N-2.8, U4 MCP3422Axx-xSN

Commit message: bom updats after the PCB assembly
Parts:
- D1, D2: value PMEG4050CEPX -> PMEG3050CEP
- R1: value 27k -> 68k
- R10: value 2k -> 20k
- R11, R12: value 3K3 -> 10K
Changed lines of the file:
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@@
 			)
 		)
-		(property "Value" "3K3"
+		(property "Value" "10K"
 			(at 112.014 163.068 90)
 			(effects
@@
 			)
 		)
-		(property "Value" "27k"
+		(property "Value" "68k"
 			(at 190.5 101.6001 0)
 			(effects
@@
 		(on_board yes)
 		(dnp no)
-		(fields_autoplaced yes)
 		(property "Reference" "C5"
-			(at 124.46 105.4099 0)
+			(at 114.554 105.918 0)
 			(effects
 				(font
@@
 		)
 		(property "Value" "2.2n"
-			(at 124.46 107.9499 0)
+			(at 114.554 103.378 0)
 			(effects
 				(font
@@
 			)
 		)
-		(property "Value" "PMEG4050CEPX"
+		(property "Value" "PMEG3050CEP"
 			(at 53.6575 88.9 0)
 			(effects
@@
 		(dnp no)
 		(property "Reference" "R12"
-			(at 113.284 163.068 90)
+			(at 117.856 163.068 90)
 			(effects
 				(font
@@
 			)
 		)
-		(property "Value" "3K3"
+		(property "Value" "10K"
 			(at 115.824 163.068 90)
 			(effects
@@
 			)
 		)
-		(property "Value" "2k"
+		(property "Value" "20k"
 			(at 255.27 139.6999 0)
 			(effects
@@
 			)
 		)
-		(property "Value" "PMEG4050CEPX"
+		(property "Value" "PMEG3050CEP"
 			(at 165.1 102.5524 90)
 			(effects
@@
 		(on_board yes)
 		(dnp no)
-		(fields_autoplaced yes)
 		(property "Reference" "C19"
 			(at 245.11 104.1399 0)
@@
 		)
 		(property "Value" "10u"
-			(at 245.11 106.6799 0)
+			(at 236.728 105.664 90)
 			(effects
 				(font
